Commit message: Fixed ueye configuation.
Former-commit-id: 760b169aab27de53b1da4d7d3fab628eaf4585bb
Former-commit-id: 142818b1a0a1aebb15b70e4799c408eebaed9d1f

File: etna_workcell/urdf/mashes_workcell.xacro (robot description, xacro)
@@ -6,5 +6,5 @@
   </xacro:property>
   <xacro:property name="camera_frame">
-    <origin xyz="0.2879 -0.0399 0.1267" rpy="1.55420 0.00225 1.59185" />
+    <origin xyz="0.0555 0.1699 0.3963" rpy="-1.161231 0.274247 -2.063781" />
   </xacro:property>
   <link name="world" />
