Commit message: Moved some cell description files to aimen package.

File: etna_workcell/urdf/diode_head.xacro (robot description, xacro)
@@ -9,5 +9,5 @@
   <visual>
     <geometry>
-      <mesh filename="package://etna_workcell/meshes/head_diode/head_diode.stl" />
+      <mesh filename="package://etna_workcell/meshes/head_diode/head.stl" />
     </geometry>
     <material name="gray">

File: etna_workcell/urdf/etna_workcell.xacro (robot description, xacro)
@@ -52,5 +52,5 @@
   <visual>
     <geometry>
-      <mesh filename="package://etna_workcell/meshes/cell/cell.stl"/>
+      <mesh filename="package://aimen_workcell/meshes/cell/cell.stl"/>
     </geometry>
     <origin xyz="0 0 0" />

File: etna_workcell/urdf/fiber_head.xacro (robot description, xacro)
@@ -9,5 +9,5 @@
   <visual>
     <geometry>
-      <mesh filename="package://etna_workcell/meshes/head/head.stl"/>
+      <mesh filename="package://etna_workcell/meshes/fiber_head/head.stl"/>
     </geometry>
     <material name="gray">
